File: design_files/Angel/angel.brd (EAGLE design)
At the start: 23 x 23.5 mm, 10 parts

Commit message: adds updates and pics
Parts:
- moved R2 3.36 mm to (6.50, 18.8)
- moved R3 3.36 mm to (17.5, 18.8)
Connections:
- net VBAT: now also U$1.P$3, U$1.P$6, VBAT.1; no longer U$1.P$1, U$1.P$4, VBAT.2
Routing:
- net GND: track 0.00 -> 7.93 mm
- net VBAT: track 11.1 -> 18.1 mm
- net VCC: track 48.6 -> 51.0 mm
- net N$1: track 1.84 -> 2.04 mm, vias 0 -> 1
- net N$2: track 1.84 -> 2.04 mm, vias 0 -> 1
- net N$3: track 6.18 -> 6.07 mm, vias 0 -> 1
- net N$4: track 6.14 -> 6.19 mm, vias 0 -> 1
Other:
- outline, holes or cut-outs redrawn
